File: Power Distribution/Power Distribution.kicad_pcb (KiCad board)
At the start: 16 copper layers, 20 parts, among them IC3 PCM5102 Audio Stereo DAC

Commit message: fixed pathing
Routing:
- net (no net): track 830.5 -> 822.6 mm

Commit message: oled files
Other:
- board outline added: 61 x 88 mm
Changed lines of the file:
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@@
 		(embedded_fonts no)
+	)
+	(gr_rect
+		(start 80 24.5)
+		(end 141 112.5)
+		(stroke
+			(width 0.05)
+			(type default)
+		)
+		(fill no)
+		(layer "Edge.Cuts")
 	)
 	(gr_text "Battery"
@@
 	(segment
 		(start 105 61.5)
-		(end 109.5 61.5)
+		(end 108.5 61.5)
 		(width 0.2)
 		(layer "F.Cu")
@@
 	)
 	(segment
+		(start 109 61.5)
+		(end 109.5 61)
+		(width 0.2)
+		(layer "F.Cu")
+		(net 0)
+	)
+	(segment
 		(start 128.27 45.89)
 		(end 128.27 43.23)
@@
 	)
 	(segment
+		(start 109.5 61)
+		(end 109.5 59.14)
+		(width 0.2)
+		(layer "F.Cu")
+		(net 0)
+	)
+	(segment
 		(start 128.27 43.23)
 		(end 128.5 43)
@@
 	)
 	(segment
-		(start 109.5 61.5)
-		(end 109.5 59.14)
-		(width 0.2)
-		(layer "F.Cu")
-		(net 0)
-	)
-	(segment
 		(start 104.5 68)
 		(end 104.5 97.32)
@@
 	)
 	(segment
-		(start 109.5 61.5)
+		(start 109.5 62)
 		(end 109.5 68.25)
 		(width 0.2)
@@
 	)
 	(segment
+		(start 109 61.5)
+		(end 109.5 62)
+		(width 0.2)
+		(layer "F.Cu")
+		(net 0)
+	)
+	(segment
 		(start 118.353 73.647)
 		(end 122 73.647)
@@
 		(width 0.2)
 		(layer "F.Cu")
+		(net 0)
+	)
+	(segment
+		(start 108.5 61.5)
+		(end 109 61.5)
+		(width 0.2)
+		(layer "F.Cu")

Commit message: PCB update
Parts:
- removed the ? at (94.0, 28.5)
- removed the ? at (88.5, 28.5)
- removed the ? at (91.5, 28.5)
- removed the ? at (86.0, 28.5)
- removed the REF** at (118.0, 75.0)
- removed the REF** at (122.0, 75.0)
- added ?: , , F.Cu at (226.5, 77.5)
- added ?: , , F.Cu at (213.5, 77.5)
- added ?: , , F.Cu at (221.4, 77.5)
- added ?: , , F.Cu at (218.5, 77.5)
- added ?: , , F.Cu at (224.0, 77.5)
- added ?: , , F.Cu at (216.0, 77.5)
- added REF**: , LC709203F:1X06_ROUND_70, F.Cu at (265.5, 126.0)
- added REF**: Thermistor 10k, Thermistor 10k:RES_NCU15X_MUR-L, F.Cu at (267.5, 120.5)
- added U$19: MOUNTINGHOLE2.5, LC709203F:MOUNTINGHOLE_2.5_PLATED, F.Cu at (265.6, 136.2)
- added U$21: MOUNTINGHOLE2.5, LC709203F:MOUNTINGHOLE_2.5_PLATED, F.Cu at (265.6, 115.9)
- added UNK_HOLE_0: , LC709203F:dummyfp0, F.Cu at (250.4, 136.2)
- added UNK_HOLE_1: , LC709203F:dummyfp1, F.Cu at (250.4, 115.9)
- moved ? 136.8 mm to (243.0, 128.5)
- moved ? 136.8 mm to (255.5, 139.5)
- moved ? 136.8 mm to (258.0, 139.5)
- moved ? 136.8 mm to (243.0, 131.0)
- moved ? 136.8 mm to (240.0, 104.5)
- moved ? 136.8 mm to (245.5, 128.5)
- moved REF** 136.8 mm to (260.5, 107.5)
- moved REF** 136.8 mm to (260.5, 100.0)
- moved ? 136.8 mm to (245.5, 131.0)
- moved ? 136.8 mm to (242.5, 104.5)
- moved IC3 136.8 mm to (232.1, 94.6)
- moved REF** 136.8 mm to (254.5, 86.5)
- moved REF** 136.8 mm to (223.0, 129.0)
- moved TP4056 & MT3608 136.8 mm to (250.0, 149.0)
Routing:
- net (no net): track 822.5 -> 1051.9 mm
Other:
- outline, holes or cut-outs redrawn
- board text added: "GND"
- board text added: "INT"
- board text added: "LC709203"
- board text added: "SCL"
- board text added: "SDA"
- board text added: "Therm"
- board text added: "VIN"

Commit message: PCB
Parts:
- removed the REF** at (267.5, 120.5)
- added ?: , , F.Cu at (259.5, 122.0)
- added ?: , , F.Cu at (259.5, 124.5)
- added G***: LOGO, Logo:VisionLogo, B.Cu at (219.0, 157.5)
Routing:
- net (no net): track 1051.9 -> 1198.5 mm
Other:
- board text added: "Thermistor 10k"
